File: kicad/pcbs/polished.kicad_pcb (KiCad board)
At the start: 2 copper layers, 127.6 x 92.9 mm, 38 parts

Commit message: Generate pcb
Parts:
- removed the G*** at (97.7, -30.2) (x2)
- added G***: LOGO, graphics:unit01XXL, F.Cu at (50.9, -20.8)
- added G***: LOGO, graphics:evaLogo, F.Cu at (99.0, -39.0)
- added G***: LOGO, graphics:unit01XXL, B.Cu at (50.9, -20.8)
- added G***: LOGO, graphics:evaLogo, B.Cu at (100.6, -38.9)
Other:
- board text removed: "made by yunk"
